File: Hardware/Qwiic Micro/SparkFun_Micro_Temperature_Sensor-STTS22H.brd (EAGLE design)
At the start: 19.1 x 7.6 mm, 40 parts, among them J1 Qwiic Right Angle, U2 STTS22H

Commit message: Adds Production files for Qwiic Micro
Parts:
- moved U$9 0.13 mm to (8.59, 1.55)
Changed lines of the file:
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@@
 <element name="U$7" library="bot" package="STTS22H11" value="" x="6.096" y="3.81" smashed="yes" rot="R90"/>
 <element name="U$8" library="bot" package="STTS22H11" value="" x="8.5852" y="2.5908" smashed="yes" rot="MR0"/>
-<element name="U$9" library="bot" package="TEMP24" value="" x="8.7122" y="1.5494" smashed="yes" rot="MR0"/>
+<element name="U$9" library="bot" package="TEMP24" value="" x="8.5852" y="1.5494" smashed="yes" rot="MR0"/>
 <element name="U$11" library="bot" package="SENSOR25" value="" x="8.5852" y="0.8128" smashed="yes" rot="MR0"/>
 <element name="R5" library="SparkFun-Resistors" package="0402-TIGHT" value="15K" x="11.938" y="2.54" smashed="yes" rot="R90">
