File: Hardware/Qwiic/SparkFun_Temperature_Sensor-STTS22H.brd (EAGLE design)
At the start: 25.4 x 25.4 mm, 54 parts, among them J1 QWIIC_RIGHT_ANGLE, J2 QWIIC_RIGHT_ANGLE, U2 STTS22H

Commit message: Adds default address text
Parts:
- added U$27: (no value), top:DEF_ADDR#29
- added U$28: (no value), top:0X3C30
Changed lines of the file:
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@@
 <attribute name="VALUE" x="11.43" y="10.287" size="0.4064" layer="28" rot="MR180"/>
 </element>
-<element name="LOGO3" library="SparkFun-Aesthetics" package="SFE_LOGO_NAME_FLAME_.1" value="SFE_LOGO_NAME_FLAME.1_INCH" x="12.658725" y="21.409025" smashed="yes" rot="MR0"/>
+<element name="LOGO3" library="SparkFun-Aesthetics" package="SFE_LOGO_NAME_FLAME_.1" value="SFE_LOGO_NAME_FLAME.1_INCH" x="12.7" y="21.409025" smashed="yes" rot="MR0"/>
 <element name="J1" library="SparkFun-Connectors" package="JST04_1MM_RA" value="QWIIC_RIGHT_ANGLE" x="20.2946" y="12.7" smashed="yes" rot="R90">
 <attribute name="NAME" x="22.4536" y="11.303" size="0.6096" layer="25" font="vector" ratio="20" rot="R90"/>
@@
 <attribute name="VALUE" x="10.922" y="12.7" size="0.6096" layer="27" font="vector" ratio="20" rot="R90" align="top-center"/>
 </element>
+<element name="U$28" library="top" package="0X3C30" value="" x="19.05" y="10.16" smashed="yes" rot="MR0"/>
+<element name="U$27" library="top" package="DEF_ADDR#29" value="" x="19.05" y="11.43" smashed="yes" rot="MR0"/>
 </elements>
 <signals>

Commit message: Replaces r7 with a 57.6k resistor
Parts:
- R7: value 56k -> 57.6k
Changed lines of the file:
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@@
 <attribute name="VALUE" x="19.05" y="14.097" size="0.6096" layer="28" font="vector" ratio="20" rot="MR0" align="top-center"/>
 </element>
-<element name="R7" library="SparkFun-Resistors" package="0603" value="56k" x="15.24" y="17.78" smashed="yes" rot="R270">
+<element name="R7" library="SparkFun-Resistors" package="0603" value="57.6k" x="15.24" y="17.78" smashed="yes" rot="R270">
 <attribute name="NAME" x="16.002" y="17.78" size="0.6096" layer="25" font="vector" ratio="20" rot="R270" align="bottom-center"/>
-<attribute name="VALUE" value="56k" x="14.478" y="17.78" size="0.6096" layer="27" font="vector" ratio="20" rot="R270" align="top-center"/>
+<attribute name="PROD_ID" value="RES-15818" x="15.24" y="17.78" size="1.778" layer="27" rot="R270" display="off"/>
+<attribute name="VALUE" value="57.6k" x="14.478" y="17.78" size="0.6096" layer="27" font="vector" ratio="20" rot="R270" align="top-center"/>
 </element>
 <element name="R8" library="SparkFun-Resistors" package="0603" value="15k" x="12.7" y="17.78" smashed="yes" rot="R90">

Commit message: Adds 56k to R7
Parts:
- R7: value 57.6k -> 56k
Changed lines of the file:
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@@
 <attribute name="VALUE" x="19.05" y="14.097" size="0.6096" layer="28" font="vector" ratio="20" rot="MR0" align="top-center"/>
 </element>
-<element name="R7" library="SparkFun-Resistors" package="0603" value="57.6k" x="15.24" y="17.78" smashed="yes" rot="R270">
+<element name="R7" library="SparkFun-Resistors" package="0603" value="56k" x="15.24" y="17.78" smashed="yes" rot="R270">
 <attribute name="NAME" x="16.002" y="17.78" size="0.6096" layer="25" font="vector" ratio="20" rot="R270" align="bottom-center"/>
-<attribute name="PROD_ID" value="RES-15818" x="15.24" y="17.78" size="1.778" layer="27" rot="R270" display="off"/>
-<attribute name="VALUE" value="57.6k" x="14.478" y="17.78" size="0.6096" layer="27" font="vector" ratio="20" rot="R270" align="top-center"/>
+<attribute name="PROD_ID" value="RES-17211" x="15.24" y="17.78" size="1.778" layer="27" rot="R270" display="off"/>
+<attribute name="VALUE" value="56k" x="14.478" y="17.78" size="0.6096" layer="27" font="vector" ratio="20" rot="R270" align="top-center"/>
 </element>
 <element name="R8" library="SparkFun-Resistors" package="0603" value="15k" x="12.7" y="17.78" smashed="yes" rot="R90">
